File: hardware/Pressure_Mat/pressure_mat_try1.sch (EAGLE design)
At the start: 34 parts, among them IC1 MCP23017T-E_ML, U1 MUX-74HC4067

Commit message: Uploaded new Eagle schematic and board
Parts:
- added IC2, IC3, IC4, IC5, IC6, IC7, IC8: MCP23017T-E_ML, SamacSys_Parts:MCP23017T-E_ML
- added R12, R13, R14, R15, R16, R17, R18, R19, R20, R21, R22, R23, R24, R25: 4.7k, SparkFun-Resistors:4.7KOHM-0603-1/10W-1%
Connections:
- new net PIN_3: IC1.INTB, IC2.INTB, IC3.INTB, IC4.INTB, IC5.INTB, IC6.INTB, IC7.INTB, IC8.INTB
- net GND: now also IC2.A1, IC2.A2, IC2.VSS, IC3.A0, IC3.A2, IC3.VSS, IC4.A2, IC4.VSS, IC5.A0, IC5.A1, IC5.VSS, IC6.A1, IC6.VSS, IC7.A0, IC7.VSS, IC8.VSS
- net I2C$SCL: now also IC2.SCL, IC3.SCL, IC4.SCL, IC5.SCL, IC6.SCL, IC7.SCL, IC8.SCL, R13.2, R15.2, R17.2, R19.2, R21.2, R23.2, R25.2
- net I2C$SDA: now also IC2.SDA, IC3.SDA, IC4.SDA, IC5.SDA, IC6.SDA, IC7.SDA, IC8.SDA, R12.2, R14.2, R16.2, R18.2, R20.2, R22.2, R24.2
- net P$1: now also IC1.GPA0
- net P$10: now also IC1.GPB1
- net P$100: now also IC7.GPA3
- net P$101: now also IC7.GPA4
- net P$102: now also IC7.GPA5
- net P$103: now also IC7.GPA6
- net P$104: now also IC7.GPA7
- net P$105: now also IC7.GPB0
- net P$106: now also IC7.GPB1
- net P$107: now also IC7.GPB2
- net P$108: now also IC7.GPB3
- net P$109: now also IC7.GPB4
- net P$11: now also IC1.GPB2
- net P$110: now also IC7.GPB5
- net P$111: now also IC7.GPB6
- net P$112: now also IC7.GPB7
- net P$113: now also IC8.GPA0
- net P$114: now also IC8.GPA1
- net P$115: now also IC8.GPA2
- net P$116: now also IC8.GPA3
- net P$117: now also IC8.GPA4
- net P$118: now also IC8.GPA5
- net P$119: now also IC8.GPA6
- net P$12: now also IC1.GPB3
- net P$120: now also IC8.GPA7
- net P$121: now also IC8.GPB0
- net P$122: now also IC8.GPB1
- net P$123: now also IC8.GPB2
- net P$124: now also IC8.GPB3
- net P$125: now also IC8.GPB4
- net P$126: now also IC8.GPB5
- net P$127: now also IC8.GPB6
- net P$128: now also IC8.GPB7
- net P$13: now also IC1.GPB4
- net P$14: now also IC1.GPB5
- net P$15: now also IC1.GPB6
- net P$16: now also IC1.GPB7
- net P$17: now also IC2.GPA0
- net P$18: now also IC2.GPA1
- net P$19: now also IC2.GPA2
- net P$2: now also IC1.GPA1
- net P$20: now also IC2.GPA3
- net P$21: now also IC2.GPA4
- net P$22: now also IC2.GPA5
- net P$23: now also IC2.GPA6
- net P$24: now also IC2.GPA7
- net P$25: now also IC2.GPB0
- net P$26: now also IC2.GPB1
- net P$27: now also IC2.GPB2
- net P$28: now also IC2.GPB3
- net P$29: now also IC2.GPB4
- net P$3: now also IC1.GPA2
- net P$30: now also IC2.GPB5
- net P$31: now also IC2.GPB6
- net P$32: now also IC2.GPB7
- net P$33: now also IC3.GPA0
- net P$34: now also IC3.GPA1
- net P$35: now also IC3.GPA2
- net P$36: now also IC3.GPA3
- net P$37: now also IC3.GPA4
- net P$38: now also IC3.GPA5
- net P$39: now also IC3.GPA6
- net P$4: now also IC1.GPA3
- net P$40: now also IC3.GPA7
- net P$41: now also IC3.GPB0
- net P$42: now also IC3.GPB1
- net P$43: now also IC3.GPB2
- net P$44: now also IC3.GPB3
- net P$45: now also IC3.GPB4
- net P$46: now also IC3.GPB5
- net P$47: now also IC3.GPB6
- net P$48: now also IC3.GPB7
- net P$49: now also IC4.GPA0
- net P$5: now also IC1.GPA4
- net P$50: now also IC4.GPA1
- net P$51: now also IC4.GPA2
- net P$52: now also IC4.GPA3
- net P$53: now also IC4.GPA4
- net P$54: now also IC4.GPA5
- net P$55: now also IC4.GPA6
- net P$56: now also IC4.GPA7
- net P$57: now also IC4.GPB0
- net P$58: now also IC4.GPB1
- net P$59: now also IC4.GPB2
- net P$6: now also IC1.GPA5
- net P$60: now also IC4.GPB3
- net P$61: now also IC4.GPB4
- net P$62: now also IC4.GPB5
- net P$63: now also IC4.GPB6
- net P$64: now also IC4.GPB7
- net P$65: now also IC5.GPA0
- net P$66: now also IC5.GPA1
- net P$67: now also IC5.GPA2
- net P$68: now also IC5.GPA3
- net P$69: now also IC5.GPA4
- net P$7: now also IC1.GPA6
- net P$70: now also IC5.GPA5
- net P$71: now also IC5.GPA6
- net P$72: now also IC5.GPA7
- net P$73: now also IC5.GPB0
- net P$74: now also IC5.GPB1
- net P$75: now also IC5.GPB2
- net P$76: now also IC5.GPB3
- net P$77: now also IC5.GPB4
- net P$78: now also IC5.GPB5
- net P$79: now also IC5.GPB6
- net P$8: now also IC1.GPA7
- net P$80: now also IC5.GPB7
- net P$81: now also IC6.GPA0
- net P$82: now also IC6.GPA1
- net P$83: now also IC6.GPA2
- net P$84: now also IC6.GPA3
- net P$85: now also IC6.GPA4
- net P$86: now also IC6.GPA5
- net P$87: now also IC6.GPA6
- net P$88: now also IC6.GPA7
- net P$89: now also IC6.GPB0
- net P$9: now also IC1.GPB0
- net P$90: now also IC6.GPB1
- net P$91: now also IC6.GPB2
- net P$92: now also IC6.GPB3
- net P$93: now also IC6.GPB4
- net P$94: now also IC6.GPB5
- net P$95: now also IC6.GPB6
- net P$96: now also IC6.GPB7
- net P$97: now also IC7.GPA0
- net P$98: now also IC7.GPA1
- net P$99: now also IC7.GPA2
- net VCC: now also IC2.!RESET, IC2.A0, IC2.VDD, IC3.!RESET, IC3.A1, IC3.VDD, IC4.!RESET, IC4.A0, IC4.A1, IC4.VDD, IC5.!RESET, IC5.A2, IC5.VDD, IC6.!RESET, IC6.A0, IC6.A2, IC6.VDD, IC7.!RESET, IC7.A1, IC7.A2, IC7.VDD, IC8.!RESET, IC8.A0, IC8.A1, IC8.A2, IC8.VDD, R12.1, R13.1, R14.1, R15.1, R16.1, R17.1, R18.1, R19.1, R20.1, R21.1, R22.1, R23.1, R24.1, R25.1
Other:
- moved on the sheet: B1, C2
