File: hardware/Pressure_Mat_Revised5-1-19/pressure_mat_try2.brd (EAGLE design)
At the start: 290 x 290 mm, 90 parts

Commit message: new stuff
new stuff
Parts:
- R68: value 100k -> 100
- moved C9 409.1 mm to (288.0, 260.0), turned to 90 degrees
- moved C10 402.8 mm to (288.0, 247.5), turned to 90 degrees
- moved R68 402.5 mm to (288.0, 243.5), turned to 90 degrees
- moved C8 373.9 mm to (288.0, 210.5), turned to 90 degrees
- moved C5 367.8 mm to (276.0, 226.0)
- moved C7 356.2 mm to (288.0, 184.5), turned to 90 degrees
- moved C4 339.1 mm to (274.5, 184.5)
- moved C6 307.9 mm to (287.5, 83.0), turned to 90 degrees
- moved C3 292.7 mm to (275.0, 83.0)
- moved C1 282.3 mm to (277.0, 25.5)
- moved DIGITAL_MUX4 3.54 mm to (279.5, 259.8)
- moved ADC 2.50 mm to (280.4, 245.3)
- moved ANALOG_MUX2 2.50 mm to (280.4, 184.4)
- moved ANALOG_MUX1 2.00 mm to (280.9, 82.9)
- moved DIGITAL_MUX3 2.00 mm to (281.5, 210.4)
Routing:
- net GND: track 0.00 -> 836.3 mm, vias 0 -> 13
- net 3.3V0: track 0.00 -> 585.5 mm, vias 0 -> 15
- net D3: track 0.00 -> 502.9 mm, vias 0 -> 11
- net D2: track 0.00 -> 416.5 mm, vias 0 -> 15
- net D0: track 0.00 -> 410.2 mm, vias 0 -> 15
- net I2C$SDA: track 0.00 -> 406.8 mm, vias 0 -> 7
- net D1: track 0.00 -> 395.3 mm, vias 0 -> 11
- net I2C$SCL: track 0.00 -> 386.5 mm, vias 0 -> 7
- net PIN_3: track 0.00 -> 323.9 mm, vias 0 -> 12
- net EN0: track 0.00 -> 279.2 mm, vias 0 -> 7
- net A_MUX0_OUT: track 0.00 -> 275.3 mm, vias 0 -> 4
- net CS: track 0.00 -> 193.7 mm, vias 0 -> 5
- net CLK: track 0.00 -> 187.0 mm, vias 0 -> 4
- net MOSI: track 0.00 -> 182.1 mm, vias 0 -> 2
- net MISO: track 0.00 -> 176.9 mm, vias 0 -> 2
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Other:
- board text added: "100"
- board text added: "10k"
- board text added: "MCP23017"
- board text added: "MUX"
- board text added: "R68"
